Commit message: ajuste comunicação arduino

File: description/ros2_control/diffbot.ros2_control.xacro (robot description, xacro)
@@ -8,8 +8,8 @@
         <param name="right_wheel_name">right_wheel_joint</param>
         <param name="loop_rate">30</param>
-        <param name="device">/dev/serial/by-path/platform-fd500000.pcie-pci-0000:01:00.0-usb-0:1.3:1.0-port0</param>
+        <param name="device">/dev/ttyUSB0</param> <!--/dev/serial/by-path/platform-fd500000.pcie-pci-0000:01:00.0-usb-0:1.3:1.0-port0</param>-->
         <param name="baud_rate">57600</param>
         <param name="timeout_ms">1000</param>
-        <param name="enc_counts_per_rev">3436</param>
+        <param name="enc_counts_per_rev">2000</param>
         <param name="pid_p">20</param>
         <param name="pid_d">12</param>

File: description/urdf/diffbot_description.urdf.xacro (robot description, xacro)
@@ -4,13 +4,13 @@
   <!-- Constants for robot dimensions -->
   <xacro:property name="PI" value="3.1415926535897931"/>
-  <xacro:property name="base_mass" value="0.3" /> <!-- arbitrary value for base mass -->
-  <xacro:property name="base_width" value="0.1" />
-  <xacro:property name="base_length" value="0.1" />
-  <xacro:property name="base_height" value="0.05" />
-  <xacro:property name="wheel_mass" value="0.3" /> <!-- arbitrary value for wheel mass -->
-  <xacro:property name="wheel_len" value="0.020" />
-  <xacro:property name="wheel_radius" value="0.015" />
-  <xacro:property name="caster_wheel_mass" value="0.1" /> <!-- arbitrary value for caster wheel mass -->
-  <xacro:property name="caster_wheel_radius" value="0.015" />
+  <xacro:property name="base_mass" value="6.000" /> <!-- arbitrary value for base mass -->
+  <xacro:property name="base_width" value="0.330" />
+  <xacro:property name="base_length" value="0.442" />
+  <xacro:property name="base_height" value="0.100" />
+  <xacro:property name="wheel_mass" value="0.525" /> <!-- arbitrary value for wheel mass -->
+  <xacro:property name="wheel_len" value="0.027" />
+  <xacro:property name="wheel_radius" value="0.050" />
+  <xacro:property name="caster_wheel_mass" value="0.100" /> <!-- arbitrary value for caster wheel mass -->
+  <xacro:property name="caster_wheel_radius" value="0.030" />
   <xacro:property name="z_offset" value="-${base_height/2}" /> <!-- Space btw top of beam and the each joint -->
   <!-- Base Link -->
@@ -19,5 +19,5 @@
       <origin xyz="0 0 0" rpy="0 0 0"/>
       <geometry>
-        <box size="${base_width} ${base_length} ${base_height}"/>
+        <box size="${base_length} ${base_width} ${base_height}"/>
       </geometry>
     </collision>
@@ -25,7 +25,7 @@
       <origin xyz="0 0 ${base_height/2}" rpy="0 0 0"/>
       <geometry>
-        <box size="${base_width} ${base_length} ${base_height}"/>
+        <box size="${base_length} ${base_width} ${base_height}"/>
       </geometry>
-      <material name="orange"/>
+      <material name="black"/>
     </visual>
     <inertial>
@@ -105,5 +105,5 @@
       <origin xyz="${base_width/2 - caster_wheel_radius} 0 ${z_offset}" rpy="0 0 0"/>
     </joint>
-    <!-- caster frontal wheel Link -->
+    <!-- caster frontal wheel Link-->
     <link name="${prefix}caster_frontal_wheel">
       <collision>
